File: e18_cc2652p.brd (EAGLE design)
At the start: 23.4 x 14.8 mm, 44 parts, among them IC3 CC2652R1FRGZ, Q1 32.768kHz, U1 MX25R8035FZUIL0, Y1 Q22FA12800150

Commit message: Add files via upload
Parts:
- C10, C3, C9: value CAP0402 -> 1pf
- C19, C4: value CAP0402 -> 12pf
- C20, C22: value CAP0402 -> 6.8pf
- C21, C23: value CAP0402 -> 1.8pf
- L3, L4: value IND0402IND0402 -> 2.4uH
- L5, L6: value IND0402IND0402 -> 2uH
- moved C11 0.18 mm to (12.0, 13.5)
- moved C6 0.11 mm to (15.6, 9.69)
- moved G 0.10 mm to (17.6, 9.53)
- moved C7 0.09 mm to (14.6, 10.2)
- moved R5 0.08 mm to (16.6, 9.70)
Routing:
- net GND: track 5.61 -> 6.84 mm, vias 79 -> 81
- net VDDR: track 6.72 -> 7.92 mm
- net VCC: track 13.5 -> 14.4 mm
- net 29: track 9.52 -> 8.63 mm
- net 28: track 8.47 -> 7.64 mm
- net N$11: track 7.63 -> 8.28 mm
- net 27: track 7.37 -> 6.76 mm
- net 26: track 6.77 -> 6.25 mm

Commit message: Add files via upload
Parts:
- moved C22 0.31 mm to (12.2, 1.80)
- moved C20 0.30 mm to (8.23, 1.63)
- moved Y1 0.29 mm to (10.2, 1.72)
- moved C13 0.27 mm to (7.21, 1.65)
Routing:
- net N$15: track 4.02 -> 4.70 mm

Commit message: Add files via upload
Parts:
- moved U$1 16.1 mm to (11.0, 18.2), turned to 0 degrees
- moved R2 16.1 mm to (1.04, 16.7), turned to 0 degrees
- moved R4 14.8 mm to (2.81, 16.7), turned to 0 degrees
- moved G 14.7 mm to (5.32, 17.5), turned to 0 degrees
- moved C21 14.1 mm to (11.0, 16.7), turned to 89.6 degrees
- moved X1 14.1 mm to (13.6, 15.4), turned to 180 degrees
- moved L6 13.9 mm to (8.48, 17.1), turned to 0 degrees
- moved C19 13.7 mm to (9.96, 16.7), turned to 270 degrees
- moved R5 13.6 mm to (4.75, 16.3), turned to 0 degrees
- moved U1 13.1 mm to (1.84, 14.6), turned to 180 degrees
- moved C23 13.0 mm to (11.0, 15.8), turned to 270 degrees
- moved J3 12.9 mm to (0.02, 2.10), turned to 90 degrees
- moved J1 12.8 mm to (14.9, 2.13), turned to 90 degrees
- moved J2 12.4 mm to (3.00, -0.15), turned to 0 degrees
- moved C2 11.9 mm to (2.06, 0.96), turned to 180 degrees
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Routing:
- net GND: track 6.84 -> 5.86 mm, vias 81 -> 82
- net X32K_Q1: track 3.75 -> 2.78 mm
- net VDDR: track 7.92 -> 7.04 mm
- net CS: track 21.3 -> 20.5 mm
Other:
- board size 23.4 x 14.8 mm -> 14.8 x 23.4 mm
- board text added: "DIO16"
- board text added: "DIO17"
- board text added: "RESET"
- board text added: "RX/DIO12"
- board text added: "SBL/DIO15"
- board text added: "TX/DIO13"
- board text removed: "DIO12"
- board text removed: "DIO13"
- board text removed: "DIO15"
- board text removed: "RST"
- board text removed: "TDI"
- board text removed: "TDO"

Commit message: Add files via upload
Parts:
- added C24: 100n, ok-discretes-dev:_PKG_C_0402
Connections:
- net GND: now also C24.1
- net VCC: now also C24.2
Routing:
- net VCC: track 14.3 -> 15.5 mm
- net GND: track 5.86 -> 5.71 mm, vias 82 -> 80

Commit message: Add files via upload
Parts:
- moved R3 19.1 mm to (2.83, 17.6), turned to 0 degrees
- moved R5 18.1 mm to (13.5, 0.51)
- moved G 17.5 mm to (12.5, 1.59), turned to 180 degrees
- moved C24 1.78 mm to (1.03, 17.6), turned to 0 degrees
- moved C15 0.67 mm to (11.5, 3.12)
- moved C5 0.64 mm to (12.4, 3.11)
- moved R1 0.58 mm to (13.3, 3.11)
- moved C6 0.21 mm to (5.46, 15.1)
- moved C7 0.18 mm to (4.36, 15.1)
- moved Q1 0.15 mm to (4.89, 13.4)
- moved C16 0.11 mm to (5.64, 2.08)
- moved L2 0.11 mm to (7.62, 2.07)
- moved C14 0.10 mm to (9.61, 2.07)
- moved L1 0.10 mm to (2.48, 3.05)
- moved C1 0.10 mm to (2.10, 1.87)
Routing:
- net 7: track 4.91 -> 20.6 mm, vias 0 -> 2
- net N$11: track 8.28 -> 4.29 mm
- net CLK: track 10.8 -> 8.52 mm
- net CS: track 20.5 -> 18.6 mm
- net GND: track 5.71 -> 4.48 mm, vias 80 -> 87
- net VDDS: track 15.2 -> 16.2 mm
- net 28: track 7.64 -> 6.86 mm
- net 29: track 8.65 -> 7.87 mm
- net 27: track 6.76 -> 6.17 mm
- net 24: track 6.95 -> 7.47 mm
- net TMS: track 5.24 -> 5.57 mm, vias 0 -> 1

Commit message: Add files via upload
Parts:
- moved R5 2.20 mm to (11.6, 1.61)
- moved C15 1.40 mm to (10.1, 3.19)
- moved C5 1.39 mm to (11.0, 3.19)
- moved R1 1.31 mm to (12.0, 3.19)
- moved G 1.17 mm to (13.3, 2.49), turned to 90 degrees
- moved C2 1.06 mm to (3.08, 1.38), turned to 90 degrees
- moved C16 1.06 mm to (4.58, 2.07)
- moved L2 1.04 mm to (6.58, 2.07)
- moved C14 1.04 mm to (8.58, 2.07)
- moved C1 0.49 mm to (2.09, 1.38), turned to 90 degrees
- moved L1 0.41 mm to (2.07, 3.05)
Routing:
- net RESET: track 17.0 -> 15.8 mm
- net 7: track 20.6 -> 19.5 mm
- net VDDS: track 16.2 -> 15.3 mm
- net 23: track 8.08 -> 7.20 mm
- net VCC: track 15.8 -> 16.4 mm, vias 5 -> 6
- net DCDC_SW: track 2.08 -> 2.61 mm
- net GND: track 4.48 -> 4.57 mm, vias 87 -> 88
Other:
- board text added: "G"

Commit message: Add files via upload
Routing:
- net 22: track 9.16 -> 7.05 mm
- net 7: track 19.5 -> 18.3 mm
- net 21: track 8.14 -> 7.24 mm
- net 19: track 7.25 -> 7.84 mm
- net CS: track 18.6 -> 18.1 mm
- net GND: track 4.57 -> 4.51 mm, vias 88 -> 86

Commit message: Add files via upload
Routing:
- net VDDS: track 15.4 -> 16.6 mm
- net GND: vias 86 -> 85
