File: e18_cc2652p.brd (EAGLE design)
At the start: 14.8 x 23.4 mm, 45 parts, among them IC3 CC2652R1FRGZ, Q1 32.768kHz, U1 MX25R8035FZUIL0, Y1 Q22FA12800150

Commit message: Add files via upload
Parts:
- removed C21, C23: 1.8pf, discretes-dev:CAPC1005X40N
- added R6, R7: 0, ok-discretes-dev:_PKG_C_0402
- C19: value 12pf -> 2.2pf
Connections:
- net N$6: now also R7.2, X1.3; no longer C21.2, U$1.P$1, U$1.P$10, U$1.P$11, U$1.P$12, U$1.P$13, U$1.P$14, U$1.P$15, U$1.P$16, U$1.P$17, U$1.P$18, U$1.P$2, U$1.P$3, U$1.P$4, U$1.P$5, U$1.P$6, U$1.P$7, U$1.P$8, U$1.P$9, U$1.SIGNAL
- net N$7: now also R6.1, R7.1; no longer C21.1, C23.1
- net N$8: now also R6.2, U$1.P$1, U$1.P$10, U$1.P$11, U$1.P$12, U$1.P$13, U$1.P$14, U$1.P$15, U$1.P$16, U$1.P$17, U$1.P$18, U$1.P$2, U$1.P$3, U$1.P$4, U$1.P$5, U$1.P$6, U$1.P$7, U$1.P$8, U$1.P$9, U$1.SIGNAL; no longer C23.2, X1.3
Routing:
- net N$8: track 0.98 -> 36.9 mm
- net N$6: track 33.1 -> 0.97 mm

Commit message: Add files via upload
Parts:
- moved R2 0.49 mm to (1.02, 16.2)
- moved R4 0.48 mm to (2.80, 16.2)
- moved R3 0.43 mm to (2.80, 17.2)
- moved C24 0.42 mm to (1.03, 17.2)
- moved U1 0.27 mm to (1.92, 14.4)
Routing:
- net VCC: track 16.4 -> 21.0 mm
- net GND: track 4.51 -> 2.79 mm, vias 85 -> 92
- net N$11: track 4.17 -> 5.80 mm
- net CS: track 18.1 -> 17.0 mm
- net MISO: track 6.29 -> 7.27 mm
- net CLK: track 8.70 -> 8.14 mm

Commit message: Add files via upload
Parts:
- removed R6, R7: 0, ok-discretes-dev:_PKG_C_0402
- added C21: 2.2pf, discretes-dev:CAPC1005X40N
- moved L6 1.33 mm to (9.47, 16.2)
- moved C19 1.10 mm to (11.1, 16.7), turned to 90 degrees
- moved C10 0.11 mm to (7.00, 15.8)
- moved L5 0.11 mm to (8.00, 15.8)
Connections:
- removed net N$8: R6.2, U$1.P$1, U$1.P$10, U$1.P$11, U$1.P$12, U$1.P$13, U$1.P$14, U$1.P$15, U$1.P$16, U$1.P$17, U$1.P$18, U$1.P$2, U$1.P$3, U$1.P$4, U$1.P$5, U$1.P$6, U$1.P$7, U$1.P$8, U$1.P$9, U$1.SIGNAL
- net N$5: now also C21.1
- net N$6: now also C21.2; no longer R7.2
- net N$7: now also U$1.P$1, U$1.P$10, U$1.P$11, U$1.P$12, U$1.P$13, U$1.P$14, U$1.P$15, U$1.P$16, U$1.P$17, U$1.P$18, U$1.P$2, U$1.P$3, U$1.P$4, U$1.P$5, U$1.P$6, U$1.P$7, U$1.P$8, U$1.P$9, U$1.SIGNAL; no longer R6.1, R7.1
Routing:
- net N$8: track 36.9 -> 0.00 mm
- net N$7: track 1.13 -> 32.7 mm

Commit message: Add files via upload
Parts:
- moved L5 0.26 mm to (8.25, 15.8)
- moved C10 0.21 mm to (7.21, 15.8)
- moved L6 0.20 mm to (9.67, 16.2)
Routing:
- net GND: vias 92 -> 96

Commit message: Add files via upload
Parts:
- moved C10 0.18 mm to (7.31, 15.7)
- moved L5 0.18 mm to (8.35, 15.7)
- moved L6 0.16 mm to (9.72, 16.1)
Routing:
- net GND: vias 96 -> 95

Commit message: Add files via upload
Parts:
- moved C19 0.45 mm to (11.1, 17.1)
- moved C21 0.45 mm to (11.1, 16.3)
Routing:
- net N$7: track 32.7 -> 33.4 mm
