File: e18_cc2652p.sch (EAGLE design)
At the start: 44 parts, among them IC3 CC2652R1FRGZ, Q1 32.768kHz, U1 MX25R8035FZUIL0, Y1 Q22FA12800150

Commit message: Add files via upload
Parts:
- C10, C3, C9: value CAP0402 -> 1pf
- C19, C4: value CAP0402 -> 12pf
- C20, C22: value CAP0402 -> 6.8pf
- C21, C23: value CAP0402 -> 1.8pf
- L3, L4: value IND0402IND0402 -> 2.4uH
- L5, L6: value IND0402IND0402 -> 2uH
Changed lines of the file:
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@@
 <part name="P+6" library="supply1" library_urn="urn:adsk.eagle:library:371" deviceset="VCC" device=""/>
 <part name="GND26" library="supply1" library_urn="urn:adsk.eagle:library:371" deviceset="GND" device=""/>
-<part name="L3" library="discretes-dev" deviceset="IND0402" device="IND0402"/>
-<part name="C3" library="discretes-dev" deviceset="CAP0402" device=""/>
-<part name="C4" library="discretes-dev" deviceset="CAP0402" device=""/>
-<part name="C9" library="discretes-dev" deviceset="CAP0402" device=""/>
-<part name="C10" library="discretes-dev" deviceset="CAP0402" device=""/>
-<part name="C19" library="discretes-dev" deviceset="CAP0402" device=""/>
-<part name="C21" library="discretes-dev" deviceset="CAP0402" device=""/>
+<part name="L3" library="discretes-dev" deviceset="IND0402" device="IND0402" value="2.4uH"/>
+<part name="C3" library="discretes-dev" deviceset="CAP0402" device="" value="1pf"/>
+<part name="C4" library="discretes-dev" deviceset="CAP0402" device="" value="12pf"/>
+<part name="C9" library="discretes-dev" deviceset="CAP0402" device="" value="1pf"/>
+<part name="C10" library="discretes-dev" deviceset="CAP0402" device="" value="1pf"/>
+<part name="C19" library="discretes-dev" deviceset="CAP0402" device="" value="12pf"/>
+<part name="C21" library="discretes-dev" deviceset="CAP0402" device="" value="1.8pf"/>
 <part name="GND3" library="supply1" library_urn="urn:adsk.eagle:library:371" deviceset="GND" device=""/>
 <part name="GND4" library="supply1" library_urn="urn:adsk.eagle:library:371" deviceset="GND" device=""/>
 <part name="GND5" library="supply1" library_urn="urn:adsk.eagle:library:371" deviceset="GND" device=""/>
-<part name="L4" library="discretes-dev" deviceset="IND0402" device="IND0402"/>
-<part name="L5" library="discretes-dev" deviceset="IND0402" device="IND0402"/>
-<part name="L6" library="discretes-dev" deviceset="IND0402" device="IND0402"/>
-<part name="C20" library="discretes-dev" deviceset="CAP0402" device=""/>
-<part name="C22" library="discretes-dev" deviceset="CAP0402" device=""/>
+<part name="L4" library="discretes-dev" deviceset="IND0402" device="IND0402" value="2.4uH"/>
+<part name="L5" library="discretes-dev" deviceset="IND0402" device="IND0402" value="2uH"/>
+<part name="L6" library="discretes-dev" deviceset="IND0402" device="IND0402" value="2uH"/>
+<part name="C20" library="discretes-dev" deviceset="CAP0402" device="" value="6.8pf"/>
+<part name="C22" library="discretes-dev" deviceset="CAP0402" device="" value="6.8pf"/>
 <part name="GND6" library="supply1" library_urn="urn:adsk.eagle:library:371" deviceset="GND" device=""/>
 <part name="GND20" library="supply1" library_urn="urn:adsk.eagle:library:371" deviceset="GND" device=""/>
 <part name="U$1" library="SparkFun-RF2" deviceset="ANTENNA-GROUNDED-BLE" device=""/>
 <part name="X1" library="adafruit" deviceset="ANTENNA_U.FL" device="" package3d_urn="urn:adsk.eagle:package:6240943/1"/>
-<part name="C23" library="discretes-dev" deviceset="CAP0402" device=""/>
+<part name="C23" library="discretes-dev" deviceset="CAP0402" device="" value="1.8pf"/>
 <part name="J1" library="SparkFun-Connectors" deviceset="CONN_11" device="1X8-1.27MM" package3d_urn="urn:adsk.eagle:package:38254/1"/>
 <part name="J2" library="SparkFun-Connectors" deviceset="CONN_11" device="1X8-1.27MM" package3d_urn="urn:adsk.eagle:package:38254/1"/>

Commit message: Add files via upload
Parts:
- added C24: 100n, ok-discretes-dev:CAP-0402
Connections:
- net GND: now also C24.1
- net VCC: now also C24.2
Changed lines of the file:
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@@
 <part name="R5" library="ok-discretes-dev" deviceset="RES" device="-0402" value="4.7K"/>
 <part name="GND21" library="supply1" library_urn="urn:adsk.eagle:library:371" deviceset="GND" device=""/>
+<part name="C24" library="ok-discretes-dev" deviceset="CAP" device="-0402" value="100n"/>
+<part name="GND22" library="supply1" library_urn="urn:adsk.eagle:library:371" deviceset="GND" device=""/>
 </parts>
 <sheets>
@@
 <instance part="GND21" gate="1" x="104.14" y="40.64" smashed="yes">
 <attribute name="VALUE" x="101.6" y="38.1" size="1.778" layer="96"/>
+</instance>
+<instance part="C24" gate="A" x="12.7" y="15.24" smashed="yes" rot="R90">
+<attribute name="NAME" x="9.017" y="17.2974" size="1.778" layer="95" rot="R180"/>
+<attribute name="VALUE" x="9.017" y="14.7574" size="1.778" layer="96" rot="R180"/>
+</instance>
+<instance part="GND22" gate="1" x="12.7" y="7.62" smashed="yes">
+<attribute name="VALUE" x="10.16" y="5.08" size="1.778" layer="96"/>
 </instance>
 </instances>
@@
 <pinref part="GND21" gate="1" pin="GND"/>
 </segment>
+<segment>
+<pinref part="C24" gate="A" pin="1"/>
+<pinref part="GND22" gate="1" pin="GND"/>
+<wire x1="12.7" y1="12.7" x2="12.7" y2="10.16" width="0.1524" layer="91"/>
+</segment>
 </net>
 <net name="VCC" class="0">
@@
 <segment>
 <pinref part="U1" gate="G$1" pin="VCC"/>
-<wire x1="15.24" y1="20.32" x2="7.62" y2="20.32" width="0.1524" layer="91"/>
+<wire x1="15.24" y1="20.32" x2="12.7" y2="20.32" width="0.1524" layer="91"/>
 <label x="7.62" y="20.32" size="1.778" layer="95"/>
-</segment>
-<segment>
+<pinref part="C24" gate="A" pin="2"/>
+<wire x1="12.7" y1="20.32" x2="7.62" y2="20.32" width="0.1524" layer="91"/>
+<wire x1="12.7" y1="17.78" x2="12.7" y2="20.32" width="0.1524" layer="91"/>
+<junction x="12.7" y="20.32"/>
+</segment>
+<segment>

Commit message: Add files via upload
Parts:
- removed C21, C23: 1.8pf, discretes-dev:CAP0402
- added R6, R7: 0, ok-discretes-dev:RES-0402
- C19: value 12pf -> 2.2pf
Connections:
- net N$6: now also R7.2, X1.SIGNAL; no longer C21.2, U$1.SIGNAL
- net N$7: now also R6.1, R7.1; no longer C21.1, C23.1
- net N$8: now also R6.2, U$1.SIGNAL; no longer C23.2, X1.SIGNAL
Changed lines of the file:
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@@
 <part name="C9" library="discretes-dev" deviceset="CAP0402" device="" value="1pf"/>
 <part name="C10" library="discretes-dev" deviceset="CAP0402" device="" value="1pf"/>
-<part name="C19" library="discretes-dev" deviceset="CAP0402" device="" value="12pf"/>
-<part name="C21" library="discretes-dev" deviceset="CAP0402" device="" value="1.8pf"/>
+<part name="C19" library="discretes-dev" deviceset="CAP0402" device="" value="2.2pf"/>
 <part name="GND3" library="supply1" library_urn="urn:adsk.eagle:library:371" deviceset="GND" device=""/>
 <part name="GND4" library="supply1" library_urn="urn:adsk.eagle:library:371" deviceset="GND" device=""/>
@@
 <part name="U$1" library="SparkFun-RF2" deviceset="ANTENNA-GROUNDED-BLE" device=""/>
 <part name="X1" library="adafruit" deviceset="ANTENNA_U.FL" device="" package3d_urn="urn:adsk.eagle:package:6240943/1"/>
-<part name="C23" library="discretes-dev" deviceset="CAP0402" device="" value="1.8pf"/>
 <part name="J1" library="SparkFun-Connectors" deviceset="CONN_11" device="1X8-1.27MM" package3d_urn="urn:adsk.eagle:package:38254/1"/>
 <part name="J2" library="SparkFun-Connectors" deviceset="CONN_11" device="1X8-1.27MM" package3d_urn="urn:adsk.eagle:package:38254/1"/>
@@
 <part name="C24" library="ok-discretes-dev" deviceset="CAP" device="-0402" value="100n"/>
 <part name="GND22" library="supply1" library_urn="urn:adsk.eagle:library:371" deviceset="GND" device=""/>
+<part name="R6" library="ok-discretes-dev" deviceset="RES" device="-0402" value="0"/>
+<part name="R7" library="ok-discretes-dev" deviceset="RES" device="-0402" value="0"/>
 </parts>
 <sheets>
@@
 <attribute name="NAME" x="285.369" y="75.184" size="1.778" layer="95" font="vector"/>
 </instance>
-<instance part="C21" gate="G$1" x="297.18" y="71.12" smashed="yes" rot="R90">
-<attribute name="NAME" x="295.529" y="72.644" size="1.778" layer="95" font="vector" rot="R90"/>
-</instance>
 <instance part="GND3" gate="1" x="213.36" y="45.72" smashed="yes">
 <attribute name="VALUE" x="210.82" y="43.18" size="1.778" layer="96"/>
@@
 <attribute name="VALUE" x="309.88" y="71.12" size="1.27" layer="96" rot="R180"/>
 </instance>
-<instance part="C23" gate="G$1" x="297.18" y="60.96" smashed="yes" rot="R90">
-<attribute name="NAME" x="295.529" y="62.484" size="1.778" layer="95" font="vector" rot="R90"/>
-</instance>
 <instance part="J1" gate="G$1" x="261.62" y="27.94" smashed="yes">
 <attribute name="VALUE" x="256.54" y="15.494" size="1.778" layer="96" font="vector"/>
@@
 <instance part="GND22" gate="1" x="12.7" y="7.62" smashed="yes">
 <attribute name="VALUE" x="10.16" y="5.08" size="1.778" layer="96"/>
+</instance>
+<instance part="R6" gate="G$1" x="297.18" y="71.12" smashed="yes">
+<attribute name="NAME" x="295.6814" y="68.58" size="1.778" layer="95"/>
+<attribute name="VALUE" x="297.942" y="73.66" size="1.778" layer="96" rot="R180"/>
+</instance>
+<instance part="R7" gate="G$1" x="297.18" y="60.96" smashed="yes">
+<attribute name="NAME" x="295.6814" y="58.42" size="1.778" layer="95"/>
+<attribute name="VALUE" x="297.942" y="63.5" size="1.778" layer="96" rot="R180"/>
 </instance>
 </instances>
@@
 </segment>
 </net>
-<net name="N$6" class="0">
-<segment>
-<pinref part="C21" gate="G$1" pin="2"/>
-<pinref part="U$1" gate="G$1" pin="SIGNAL"/>
-<wire x1="300.99" y1="71.12" x2="304.8" y2="71.12" width="0.1524" layer="91"/>
-</segment>
-</net>
 <net name="N$7" class="0">
 <segment>
-<pinref part="C21" gate="G$1" pin="1"/>
 <pinref part="C19" gate="G$1" pin="2"/>
 <wire x1="290.83" y1="71.12" x2="292.1" y2="71.12" width="0.1524" layer="91"/>
-<wire x1="292.1" y1="71.12" x2="293.37" y2="71.12" width="0.1524" layer="91"/>
 <wire x1="292.1" y1="71.12" x2="292.1" y2="60.96" width="0.1524" layer="91"/>
+<pinref part="R6" gate="G$1" pin="1"/>
+<wire x1="294.64" y1="71.12" x2="292.1" y2="71.12" width="0.1524" layer="91"/>
 <junction x="292.1" y="71.12"/>
-<pinref part="C23" gate="G$1" pin="1"/>
-<wire x1="292.1" y1="60.96" x2="293.37" y2="60.96" width="0.1524" layer="91"/>
-</segment>
-</net>
-<net name="N$8" class="0">
-<segment>
-<pinref part="C23" gate="G$1" pin="2"/>
-<pinref part="X1" gate="G$1" pin="SIGNAL"/>
-<wire x1="300.99" y1="60.96" x2="302.26" y2="60.96" width="0.1524" layer="91"/>
+<pinref part="R7" gate="G$1" pin="1"/>
+<wire x1="294.64" y1="60.96" x2="292.1" y2="60.96" width="0.1524" layer="91"/>
 </segment>
 </net>
@@
 </segment>
 </net>
+<net name="N$6" class="0">
+<segment>
+<pinref part="X1" gate="G$1" pin="SIGNAL"/>
+<pinref part="R7" gate="G$1" pin="2"/>
+<wire x1="302.26" y1="60.96" x2="299.72" y2="60.96" width="0.1524" layer="91"/>
+</segment>
+</net>
+<net name="N$8" class="0">
+<segment>
+<pinref part="U$1" gate="G$1" pin="SIGNAL"/>
+<pinref part="R6" gate="G$1" pin="2"/>
+<wire x1="304.8" y1="71.12" x2="299.72" y2="71.12" width="0.1524" layer="91"/>
+</segment>
+</net>

Commit message: Add files via upload
Parts:
- removed R6, R7: 0, ok-discretes-dev:RES-0402
- added C21: 2.2pf, discretes-dev:CAP0402
Connections:
- removed net N$8: R6.2, U$1.SIGNAL
- net N$5: now also C21.1
- net N$6: now also C21.2; no longer R7.2
- net N$7: now also U$1.SIGNAL; no longer R6.1, R7.1
Other:
- moved on the sheet: C19
Changed lines of the file:
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@@
 <part name="C24" library="ok-discretes-dev" deviceset="CAP" device="-0402" value="100n"/>
 <part name="GND22" library="supply1" library_urn="urn:adsk.eagle:library:371" deviceset="GND" device=""/>
-<part name="R6" library="ok-discretes-dev" deviceset="RES" device="-0402" value="0"/>
-<part name="R7" library="ok-discretes-dev" deviceset="RES" device="-0402" value="0"/>
+<part name="C21" library="discretes-dev" deviceset="CAP0402" device="" value="2.2pf"/>
 </parts>
 <sheets>
@@
 <attribute name="NAME" x="260.604" y="65.151" size="1.778" layer="95" font="vector"/>
 </instance>
-<instance part="C19" gate="G$1" x="287.02" y="71.12" smashed="yes" rot="R90">
-<attribute name="NAME" x="285.369" y="75.184" size="1.778" layer="95" font="vector"/>
+<instance part="C19" gate="G$1" x="297.18" y="71.12" smashed="yes" rot="R90">
+<attribute name="NAME" x="295.529" y="75.184" size="1.778" layer="95" font="vector"/>
 </instance>
 <instance part="GND3" gate="1" x="213.36" y="45.72" smashed="yes">
@@
 <attribute name="VALUE" x="10.16" y="5.08" size="1.778" layer="96"/>
 </instance>
-<instance part="R6" gate="G$1" x="297.18" y="71.12" smashed="yes">
-<attribute name="NAME" x="295.6814" y="68.58" size="1.778" layer="95"/>
-<attribute name="VALUE" x="297.942" y="73.66" size="1.778" layer="96" rot="R180"/>
-</instance>
-<instance part="R7" gate="G$1" x="297.18" y="60.96" smashed="yes">
-<attribute name="NAME" x="295.6814" y="58.42" size="1.778" layer="95"/>
-<attribute name="VALUE" x="297.942" y="63.5" size="1.778" layer="96" rot="R180"/>
+<instance part="C21" gate="G$1" x="297.18" y="60.96" smashed="yes" rot="R90">
+<attribute name="NAME" x="295.529" y="54.864" size="1.778" layer="95" font="vector"/>
 </instance>
 </instances>
@@
 </segment>
 </net>
-<net name="N$5" class="0">
-<segment>
-<pinref part="C19" gate="G$1" pin="1"/>
-<pinref part="L6" gate="G$1" pin="2"/>
-<wire x1="279.4" y1="71.12" x2="283.21" y2="71.12" width="0.1524" layer="91"/>
-</segment>
-</net>
-<net name="N$7" class="0">
-<segment>
-<pinref part="C19" gate="G$1" pin="2"/>
-<wire x1="290.83" y1="71.12" x2="292.1" y2="71.12" width="0.1524" layer="91"/>
-<wire x1="292.1" y1="71.12" x2="292.1" y2="60.96" width="0.1524" layer="91"/>
-<pinref part="R6" gate="G$1" pin="1"/>
-<wire x1="294.64" y1="71.12" x2="292.1" y2="71.12" width="0.1524" layer="91"/>
-<junction x="292.1" y="71.12"/>
-<pinref part="R7" gate="G$1" pin="1"/>
-<wire x1="294.64" y1="60.96" x2="292.1" y2="60.96" width="0.1524" layer="91"/>
-</segment>
-</net>
 <net name="N$9" class="0">
 <segment>
@@
 <segment>
 <pinref part="X1" gate="G$1" pin="SIGNAL"/>
-<pinref part="R7" gate="G$1" pin="2"/>
-<wire x1="302.26" y1="60.96" x2="299.72" y2="60.96" width="0.1524" layer="91"/>
-</segment>
-</net>
-<net name="N$8" class="0">
-<segment>
+<pinref part="C21" gate="G$1" pin="2"/>
+<wire x1="302.26" y1="60.96" x2="300.99" y2="60.96" width="0.1524" layer="91"/>
+</segment>
+</net>
+<net name="N$5" class="0">
+<segment>
+<pinref part="L6" gate="G$1" pin="2"/>
+<wire x1="279.4" y1="71.12" x2="287.02" y2="71.12" width="0.1524" layer="91"/>
+<pinref part="C19" gate="G$1" pin="1"/>
+<wire x1="287.02" y1="71.12" x2="293.37" y2="71.12" width="0.1524" layer="91"/>
+<wire x1="287.02" y1="71.12" x2="287.02" y2="60.96" width="0.1524" layer="91"/>
+<wire x1="287.02" y1="60.96" x2="293.37" y2="60.96" width="0.1524" layer="91"/>
+<junction x="287.02" y="71.12"/>
+<pinref part="C21" gate="G$1" pin="1"/>
+</segment>
+</net>
+<net name="N$7" class="0">
+<segment>
+<pinref part="C19" gate="G$1" pin="2"/>
 <pinref part="U$1" gate="G$1" pin="SIGNAL"/>
-<pinref part="R6" gate="G$1" pin="2"/>
-<wire x1="304.8" y1="71.12" x2="299.72" y2="71.12" width="0.1524" layer="91"/>
-</segment>
-</net>
+<wire x1="300.99" y1="71.12" x2="304.8" y2="71.12" width="0.1524" layer="91"/>
+</segment>
+</net>
