File: v1.1/e18_cc2652p.brd (EAGLE design)
At the start: 14.8 x 23.3 mm, 47 parts, among them IC3 CC2652R1FRGZ, Q1 32.768kHz, U1 MX25R8035FZUIL0, Y1 Q22FA12800150

Commit message: Add files via upload
Routing:
- net GND: vias 89 -> 91
Other:
- board size 14.8 x 23.3 mm -> 14.9 x 23.4 mm
Changed lines of the file:
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@@
 <plain>
 <text x="14.537496875" y="18.176784375" size="0.8128" layer="26" rot="MR0">JLCJLCJLCJLC</text>
-<wire x1="14.907953125" y1="-0.134753125" x2="14.907953125" y2="23.143246875" width="0.0762" layer="20"/>
-<wire x1="14.907953125" y1="23.143246875" x2="0.059153125" y2="23.143246875" width="0.0762" layer="20"/>
-<wire x1="0.059153125" y1="23.143246875" x2="0.059153125" y2="-0.134753125" width="0.0762" layer="20"/>
-<wire x1="0.059153125" y1="-0.134753125" x2="14.907953125" y2="-0.134753125" width="0.0762" layer="20"/>
+<wire x1="14.957953125" y1="-0.234753125" x2="14.957953125" y2="23.143246875" width="0.0762" layer="20"/>
+<wire x1="14.957953125" y1="23.143246875" x2="0.009153125" y2="23.143246875" width="0.0762" layer="20"/>
+<wire x1="0.009153125" y1="23.143246875" x2="0.009153125" y2="-0.234753125" width="0.0762" layer="20"/>
+<wire x1="0.009153125" y1="-0.234753125" x2="14.957953125" y2="-0.234753125" width="0.0762" layer="20"/>
 <rectangle x1="4.3453375" y1="12.975671875" x2="5.4453375" y2="13.775671875" layer="41" rot="R90"/>
 <text x="14.11966875" y="10.5450125" size="1.016" layer="26" font="vector" ratio="12" rot="SMR359.6">RESET</text>
@@
 <wire x1="11.4025875" y1="11.147971875" x2="11.3952625" y2="11.155296875" width="0.254" layer="1"/>
 <wire x1="11.3421" y1="12.1176375" x2="11.3421" y2="12.15651875" width="0.254" layer="1"/>
-<via x="10.814765625" y="12.74625625" extent="1-16" drill="0.2" diameter="0.45"/>
+<via x="10.964765625" y="12.74625625" extent="1-16" drill="0.2" diameter="0.45"/>
 <wire x1="12.554365625" y1="9.282771875" x2="12.554365625" y2="9.1912375" width="0.1524" layer="1"/>
 <via x="11.840759375" y="12.74625625" extent="1-16" drill="0.2" diameter="0.45"/>
@@
 <contactref element="C20" pad="2"/>
 <contactref element="G" pad="C"/>
-<via x="9.884159375" y="12.756759375" extent="1-16" drill="0.2" diameter="0.45"/>
+<via x="10.184159375" y="12.756759375" extent="1-16" drill="0.2" diameter="0.45"/>
 <wire x1="1.546103125" y1="4.341315625" x2="2.076471875" y2="4.341315625" width="0.3048" layer="1"/>
 <wire x1="2.076471875" y1="4.341315625" x2="2.26778125" y2="4.532625" width="0.3048" layer="1"/>
@@
 <via x="11.337953125" y="17.798146875" extent="1-16" drill="0.2" diameter="0.45"/>
 <via x="9.387953125" y="17.798146875" extent="1-16" drill="0.2" diameter="0.45"/>
-<via x="13.087953125" y="17.798146875" extent="1-16" drill="0.2" diameter="0.45"/>
+<via x="12.737953125" y="17.798146875" extent="1-16" drill="0.2" diameter="0.45"/>
 <via x="14.237953125" y="17.798146875" extent="1-16" drill="0.25" diameter="0.45"/>
 <via x="6.887009375" y="17.331440625" extent="1-16" drill="0.2" diameter="0.45"/>
@@
 <via x="12.081084375" y="13.374840625" extent="1-16" drill="0.2" diameter="0.45"/>
 <via x="9.181084375" y="14.924840625" extent="1-16" drill="0.2" diameter="0.45"/>
+<via x="9.834159375" y="12.306759375" extent="1-16" drill="0.2" diameter="0.45"/>
+<via x="13.287953125" y="17.798146875" extent="1-16" drill="0.2" diameter="0.45"/>
 </signal>
 <signal name="VCC">
@@
 <wire x1="3.158996875" y1="14.143190625" x2="2.75870625" y2="14.143190625" width="0.1524" layer="1"/>
 <wire x1="2.75870625" y1="14.143190625" x2="2.4" y2="13.784484375" width="0.1524" layer="1"/>
-<wire x1="2.4" y1="13.784484375" x2="2.4" y2="13.45" width="0.1524" layer="1"/>
-<wire x1="2.4" y1="13.45" x2="1.95" y2="13" width="0.1524" layer="1"/>
-<wire x1="1.95" y1="13" x2="1.55" y2="13" width="0.1524" layer="1"/>
+<wire x1="2.4" y1="13.784484375" x2="2.4" y2="13.5" width="0.1524" layer="1"/>
+<wire x1="2.4" y1="13.5" x2="1.9" y2="13" width="0.1524" layer="1"/>
+<wire x1="1.9" y1="13" x2="1.55" y2="13" width="0.1524" layer="1"/>
 <wire x1="1.55" y1="13" x2="1.5" y2="13" width="0.1524" layer="1"/>
 <via x="1.55" y="13" extent="1-16" drill="0.2" diameter="0.45"/>

Commit message: Add files via upload
Parts:
- IC3: value CC2652R1FRGZ -> CC2652P1FRGZ
- L3, L4: value 2.4uH -> 2.4nH
- L5, L6: value 2uH -> 2nH
- R3: value 100K -> 1M
Connections:
- net VCC: no longer C24.2, R2.2, R3.1, R4.1, U1.8
- net VDDS: now also C24.2, R2.2, R3.1, R4.1, U1.8
Routing:
- net VCC: track 21.0 -> 6.93 mm, vias 6 -> 4
- net VDDS: track 16.5 -> 30.4 mm, vias 5 -> 7
- net MISO: track 7.24 -> 5.99 mm
- net CLK: track 8.14 -> 9.20 mm
