File: v1.1/e18_cc2652p.sch (EAGLE design)
At the start: 47 parts, among them IC3 CC2652R1FRGZ, Q1 32.768kHz, U1 MX25R8035FZUIL0, Y1 Q22FA12800150

Commit message: Add files via upload
Parts:
- IC3: value CC2652R1FRGZ -> CC2652P1FRGZ
- L3, L4: value 2.4uH -> 2.4nH
- L5, L6: value 2uH -> 2nH
- R3: value 100K -> 1M
Connections:
- net VCC: no longer C24.2, R2.2, R3.1, R4.1, U1.VCC
- net VDDS: now also C24.2, R2.2, R3.1, R4.1, U1.VCC
Other:
- moved on the sheet: C24, R2, R3, R4, U1
